Commit message: car_urdf: simplify flipper collision geometry

File: car_urdf/urdf/car_urdf.urdf (robot description, URDF)
Before this commit: robot car_urdf, 25 links, 24 joints
Links:
- link left_ahead_arm: geometry collision cylinder length=0.32 radius=0.022; visual mesh filename=package://car_urdf/meshes/left_ahead_arm.STL
- link left_back_arm: geometry collision cylinder length=0.32 radius=0.022; visual mesh filename=package://car_urdf/meshes/left_back_arm.STL
- link right_ahead_arm: geometry collision cylinder length=0.32 radius=0.022; visual mesh filename=package://car_urdf/meshes/right_ahead_arm.STL
- link right_back_arm: geometry collision cylinder length=0.32 radius=0.022; visual mesh filename=package://car_urdf/meshes/right_back_arm.STL

Commit message: Tune servo scaling and update arm limits

File: car_urdf/urdf/car_urdf.urdf (robot description, URDF)
Before this commit: robot car_urdf, 25 links, 24 joints
Joints:
- joint left_gripper_finger_joint: limit lower=0.0 upper=0.044 effort=20 velocity=0.2 -> lower=-0.05 upper=0.0710 effort=20 velocity=0.2
- joint right_gripper_finger_joint: limit lower=0.0 upper=0.044 effort=20 velocity=0.2 -> lower=-0.05 upper=0.0710 effort=20 velocity=0.2
- joint wrist_pitch_joint: limit lower=-1.57 upper=2.356 effort=6 velocity=1.57 -> lower=-1.57 upper=3.09 effort=6 velocity=1.57

Commit message: Adjust elbow pitch upper limit to 3.05

File: car_urdf/urdf/car_urdf.urdf (robot description, URDF)
Before this commit: robot car_urdf, 25 links, 24 joints
Joints:
- joint elbow_pitch_joint: limit lower=-1.0 upper=2.793 effort=18 velocity=1.57 -> lower=-1.0 upper=3.05 effort=18 velocity=1.57
- joint wrist_pitch_joint: limit lower=-1.57 upper=3.09 effort=6 velocity=1.57 -> lower=-1.57 upper=2.356 effort=6 velocity=1.57

Commit message: robot_config: switch gripper controller to velocity mode

File: car_urdf/urdf/car_urdf.urdf (robot description, URDF)
Before this commit: robot car_urdf, 25 links, 24 joints
Joints:
- joint right_gripper_finger_joint: limit lower=-0.05 upper=0.0710 effort=20 velocity=0.2 -> lower=-5 upper=141 effort=20 velocity=0.2
