Commit message: checkpoint: current bringup and bridge updates

File: car_moveit_config/config/gazebo_car_urdf.urdf (robot description, URDF)
Before this commit: robot car_urdf, 23 links, 22 joints
Joints:
- joint wrist_roll_joint: axis -1 0 0 -> 0 0 1; child hands_roll_part -> handshands_course_part; limit lower=-2.356 upper=2.356 effort=6 velocity=1.57 -> lower=-7.069 upper=7.069 effort=6 velocity=1.57; origin xyz=-0.0330007142673656 -0.0330000000000009 0.0530007142674829 rpy=0 0 0 -> xyz=0.0330007142675045 0 0.0474000000000001 rpy=0 0 0; parent hands_pitch_part -> hands_roll_part
- joint wrist_yaw_joint: axis 0 0 1 -> -1 0 0; child handshands_course_part -> hands_roll_part; limit lower=-7.069 upper=7.069 effort=6 velocity=1.57 -> lower=-2.356 upper=2.356 effort=6 velocity=1.57; origin xyz=0.0330007142675045 0 0.0474000000000001 rpy=0 0 0 -> xyz=-0.0330007142673656 -0.0330000000000009 0.0530007142674829 rpy=0 0 0; parent hands_roll_part -> hands_pitch_part

File: car_urdf/urdf/car_urdf.urdf (robot description, URDF)
Before this commit: robot car_urdf, 25 links, 24 joints
Joints:
- joint wrist_roll_joint: axis -1 0 0 -> 0 0 1; child hands_roll_part -> handshands_course_part; limit lower=-2.356 upper=2.356 effort=6 velocity=1.57 -> lower=-7.069 upper=7.069 effort=6 velocity=1.57; origin xyz=-0.0330007142673656 -0.0330000000000009 0.0530007142674829 rpy=0 0 0 -> xyz=0.0330007142675045 0 0.0474000000000001 rpy=0 0 0; parent hands_pitch_part -> hands_roll_part
- joint wrist_yaw_joint: axis 0 0 1 -> -1 0 0; child handshands_course_part -> hands_roll_part; limit lower=-7.069 upper=7.069 effort=6 velocity=1.57 -> lower=-2.356 upper=2.356 effort=6 velocity=1.57; origin xyz=0.0330007142675045 0 0.0474000000000001 rpy=0 0 0 -> xyz=-0.0330007142673656 -0.0330000000000009 0.0530007142674829 rpy=0 0 0; parent hands_roll_part -> hands_pitch_part
