Commit message: feat: integrate ROS2 full system and archive ROS1 workspace
Add grouped safety and recovery, MoveIt2 control, peripheral integration, simulation, and Humble validation tools. Archive ROS1 sources and update workspace documentation and dependency pins.

File: robot_canopen_config/urdf/canopen.ros2_control.xacro (robot description, xacro)
@@ -1,5 +1,5 @@
 <?xml version="1.0"?>
 <robot xmlns:xacro="http://www.ros.org/wiki/xacro">
-  <xacro:macro name="robot_canopen_control" params="can_interface_name:=canable0 safety_domain:=robot mock:=false">
+  <xacro:macro name="robot_canopen_control" params="can_interface_name:=canable0 safety_domain:=robot mock:=false group_policy:=''">
     <ros2_control name="RobotCanopenSystem" type="system">
       <hardware>
@@ -7,4 +7,5 @@
         <xacro:unless value="${mock}"><plugin>canopen_ros2_control/RobotSystem</plugin></xacro:unless>
         <param name="safety_domain">${safety_domain}</param>
+        <xacro:if value="${group_policy != ''}"><param name="group_policy">${group_policy}</param></xacro:if>
         <param name="bus_config">$(find robot_canopen_config)/config/bus.yml</param>
         <param name="master_config">$(find robot_canopen_config)/config/master.dcf</param>

File: robot_hardware/urdf/model.urdf.xacro (robot description, xacro)
@@ -156,5 +156,5 @@
     <child link="zhua2" />
     <axis xyz="0 1 0" />
-    <limit lower="-5" upper="141" effort="20" velocity="0.2" />
+    <limit lower="-0.05" upper="0.0710" effort="20" velocity="0.2" />
     <dynamics damping="0.2" friction="0.02" />
     <mimic joint="left_gripper_finger_joint" multiplier="1" offset="0" />

File: robot_hardware/urdf/private.ros2_control.xacro (robot description, xacro)
@@ -1,5 +1,5 @@
 <?xml version='1.0' encoding='utf-8'?>
 <robot xmlns:xacro="http://www.ros.org/wiki/xacro">
-  <xacro:macro name="private_can_control" params="can_interface:=canable1 mock:=false">
+  <xacro:macro name="private_can_control" params="can_interface:=canable1 mock:=false group_policy:=''">
     <ros2_control name="CanDriverSystem" type="system">
       <hardware>
@@ -11,4 +11,5 @@
         </xacro:unless>
         <param name="safety_domain">robot</param>
+        <xacro:if value="${group_policy != ''}"><param name="group_policy">${group_policy}</param></xacro:if>
       </hardware>
       <joint name="elbow_pitch_joint">

File: robot_hardware/urdf/robot.urdf.xacro (robot description, xacro)
@@ -1,3 +1,4 @@
 <robot name="robot" xmlns:xacro="http://www.ros.org/wiki/xacro">
+ <xacro:arg name="group_policy" default=""/>
  <xacro:arg name="mock" default="false"/>
  <xacro:arg name="canopen_interface" default="canable0"/>
@@ -6,5 +7,5 @@
  <xacro:include filename="$(find robot_canopen_config)/urdf/canopen.ros2_control.xacro"/>
  <xacro:include filename="$(find robot_hardware)/urdf/private.ros2_control.xacro"/>
- <xacro:robot_canopen_control can_interface_name="$(arg canopen_interface)" mock="$(arg mock)"/>
- <xacro:private_can_control can_interface="$(arg private_interface)" mock="$(arg mock)"/>
+ <xacro:robot_canopen_control can_interface_name="$(arg canopen_interface)" mock="$(arg mock)" group_policy="$(arg group_policy)"/>
+ <xacro:private_can_control can_interface="$(arg private_interface)" mock="$(arg mock)" group_policy="$(arg group_policy)"/>
 </robot>
